File: hardware/nyx.kicad_sch (KiCad schematic)
At the start: 20 parts, among them U9 STM32F405RGTx, Y1 25MHz

Commit message: ✨ Complete footprint assignment
Parts:
- added J5: Conn_MCU_PROG, Connector_PinHeader_2.54mm:PinHeader_1x04_P2.54mm_Vertical, symbol Connector_Generic:Conn_01x04
- added SW1, SW2: SW_Push, Button_Switch_SMD:SW_SPST_B3U-1000P, symbol Switch:SW_Push
- C10, C21, C22, C25, C27, C6, C7, C8, C9: footprint (none) -> Capacitor_SMD:C_0402_1005Metric
- C23, C24, C26: footprint (none) -> Capacitor_SMD:C_0603_1608Metric
- R13, R14, R15, R16, R5, R6: footprint (none) -> Resistor_SMD:R_0603_1608Metric
- Y1: footprint (none) -> Crystal:Crystal_SMD_2016-4Pin_2.0x1.6mm
Connections:
- net +3.3V: now also SW2.2
- net BOOT: now also SW2.1
- net GND: now also J5.1 (Pin_1), SW1.1
- net RESET: now also SW1.2
- net SWDIO: now reaches U9.46 (PA13)
- net SWDIO: now also J5.2 (Pin_2)
- net SWCLK: now reaches U9.49 (PA14)
- net SWCLK: now also J5.3 (Pin_3)
- new net +5V: J5.4 (Pin_4)
Other:
- moved on the sheet: R14
